Commit message: robot llimits changed

File: movensys_manipulator_description/urdf/synustech/synustech.xacro (robot description, xacro)
@@ -30,7 +30,8 @@
     <!-- Manual - J1,J2,J4,J5,J6 +/-360 deg, J3 +/-160 deg. The full turn is
          restricted to +/-180 deg here so the IK does not pick wound-up
-         solutions (full base turns, wrist at 325 deg) for nearby poses. -->
-    <xacro:property name="lim_full"  value="${pi}"/>
-    <xacro:property name="lim_elbow" value="${160*pi/180}"/>
+         solutions (full base turns, wrist at 325 deg) for nearby poses.
+         TODO - Needs to finetune the limits-->
+    <xacro:property name="lim_full"  value="${2*pi}"/>
+    <xacro:property name="lim_elbow" value="${2*pi}"/>
     <!-- Manual - max joint velocity 120,120,180,225,225,225 deg/s. joint_vel caps them. -->
     <xacro:property name="vel_base"  value="${min(joint_vel, 120*pi/180)}"/>
